Commit message: Removed outdated URDF and old nav launch file

File: urdf/slam_nav2_bot.urdf.xacro (robot description, xacro)
@@ -27,5 +27,5 @@
         <parent link="base_footprint"/>
         <child link="base_link"/>
-        <origin xyz="0 0 0.016" rpy="0 0 4.7124"/>
+        <origin xyz="0 0 0.016" rpy="0 0 1.57"/>
     </joint>
     <link name="base_link">
